Commit message: added camera

File: ur_ws/src/Universal_Robots_ROS2_Description/urdf/ur_macro.xacro (robot description, xacro)
@@ -44,5 +44,6 @@
   <xacro:include filename="$(find ur_description)/urdf/inc/ur_transmissions.xacro" />
   <xacro:include filename="$(find ur_description)/urdf/inc/ur_common.xacro" />
-  <xacro:macro name="ur_robot" params="
+  <xacro:macro name="ur_robot"
+    params="
     name
     tf_prefix
@@ -83,311 +84,407 @@
     non_blocking_read:=false
     keep_alive_count:=2"
-    >
-    <!-- Load configuration data from the provided .yaml files -->
-    <xacro:read_model_data
-      joint_limits_parameters_file="${joint_limits_parameters_file}"
-      kinematics_parameters_file="${kinematics_parameters_file}"
-      physical_parameters_file="${physical_parameters_file}"
-      visual_parameters_file="${visual_parameters_file}"
-      force_abs_paths="${sim_gazebo or sim_ignition}"/>
-    <!-- ros2 control include -->
-    <xacro:include filename="$(find ur_description)/urdf/ur.ros2_control.xacro" />
-    <!-- ros2 control instance -->
-    <xacro:ur_ros2_control
-      name="${name}"
-      use_fake_hardware="${use_fake_hardware}"
-      initial_positions="${initial_positions}"
-      fake_sensor_commands="${fake_sensor_commands}"
-      headless_mode="${headless_mode}"
-      sim_gazebo="${sim_gazebo}"
-      sim_ignition="${sim_ignition}"
-      script_filename="${script_filename}"
-      output_recipe_filename="${output_recipe_filename}"
-      input_recipe_filename="${input_recipe_filename}"
-      tf_prefix="${tf_prefix}"
-      hash_kinematics="${kinematics_hash}"
-      robot_ip="${robot_ip}"
-      use_tool_communication="${use_tool_communication}"
-      tool_voltage="${tool_voltage}"
-      tool_parity="${tool_parity}"
-      tool_baud_rate="${tool_baud_rate}"
-      tool_stop_bits="${tool_stop_bits}"
-      tool_rx_idle_chars="${tool_rx_idle_chars}"
-      tool_tx_idle_chars="${tool_tx_idle_chars}"
-      tool_device_name="${tool_device_name}"
-      tool_tcp_port="${tool_tcp_port}"
-      reverse_port="${reverse_port}"
-      script_sender_port="${script_sender_port}"
-      reverse_ip="${reverse_ip}"
-      script_command_port="${script_command_port}"
-      trajectory_port="${trajectory_port}"
-      non_blocking_read="${non_blocking_read}"
-      keep_alive_count="${keep_alive_count}"
-      />
-    <!-- Add URDF transmission elements (for ros_control) -->
-    <!--<xacro:ur_arm_transmission prefix="${prefix}" hw_interface="${transmission_hw_interface}" />-->
-    <!-- Placeholder for ros2_control transmission which don't yet exist -->
-    <!-- links -  main serial chain -->
-    <link name="${tf_prefix}base_link"/>
-    <link name="${tf_prefix}base_link_inertia">
-      <visual>
-        <origin xyz="0 0 0" rpy="0 0 ${pi}"/>
-        <geometry>
-          <xacro:get_mesh name="base" type="visual"/>
-        </geometry>
-      </visual>
-      <collision>
-        <origin xyz="0 0 0" rpy="0 0 ${pi}"/>
-        <geometry>
-          <xacro:get_mesh name="base" type="collision"/>
-        </geometry>
-      </collision>
-      <xacro:cylinder_inertial radius="${base_inertia_radius}" length="${base_inertia_length}" mass="${base_mass}">
-        <origin xyz="0 0 0" rpy="0 0 0" />
-      </xacro:cylinder_inertial>
-    </link>
-    <link name="${tf_prefix}shoulder_link">
-      <visual>
-        <origin xyz="0 0 0" rpy="0 0 ${pi}"/>
-        <geometry>
-          <xacro:get_mesh name="shoulder" type="visual"/>
-        </geometry>
-      </visual>
-      <collision>
-        <origin xyz="0 0 0" rpy="0 0 ${pi}"/>
-        <geometry>
-          <xacro:get_mesh name="shoulder" type="collision"/>
-        </geometry>
-      </collision>
-      <xacro:cylinder_inertial radius="${shoulder_inertia_radius}" length="${shoulder_inertia_length}" mass="${shoulder_mass}">
-        <origin xyz="0 0 0" rpy="0 0 0" />
-      </xacro:cylinder_inertial>
-    </link>
-    <link name="${tf_prefix}upper_arm_link">
-      <visual>
-        <origin xyz="0 0 ${shoulder_offset}" rpy="${pi/2} 0 ${-pi/2}"/>
-        <geometry>
-          <xacro:get_mesh name="upper_arm" type="visual"/>
-        </geometry>
-      </visual>
-      <collision>
-        <origin xyz="0 0 ${shoulder_offset}" rpy="${pi/2} 0 ${-pi/2}"/>
-        <geometry>
-          <xacro:get_mesh name="upper_arm" type="collision"/>
-        </geometry>
-      </collision>
-      <xacro:cylinder_inertial radius="${upperarm_inertia_radius}" length="${upperarm_inertia_length}" mass="${upper_arm_mass}">
-        <origin xyz="${-0.5 * upperarm_inertia_length} 0.0 ${upper_arm_inertia_offset}" rpy="0 ${pi/2} 0" />
-      </xacro:cylinder_inertial>
-    </link>
-    <link name="${tf_prefix}forearm_link">
-      <visual>
-        <origin xyz="0 0 ${elbow_offset}" rpy="${pi/2} 0 ${-pi/2}"/>
-        <geometry>
-          <xacro:get_mesh name="forearm" type="visual"/>
-        </geometry>
-      </visual>
-      <collision>
-        <origin xyz="0 0 ${elbow_offset}" rpy="${pi/2} 0 ${-pi/2}"/>
-        <geometry>
-          <xacro:get_mesh name="forearm" type="collision"/>
-        </geometry>
-      </collision>
-      <xacro:cylinder_inertial radius="${forearm_inertia_radius}" length="${forearm_inertia_length}"  mass="${forearm_mass}">
-        <origin xyz="${-0.5 * forearm_inertia_length} 0.0 ${elbow_offset}" rpy="0 ${pi/2} 0" />
-      </xacro:cylinder_inertial>
-    </link>
-    <link name="${tf_prefix}wrist_1_link">
-	  <xacro:get_visual_params name="wrist_1" type="visual_offset"/>
-      <visual>
-      	<origin xyz="0 0 ${visual_params}" rpy="${pi/2} 0 0"/>
-        <geometry>
-          <xacro:get_mesh name="wrist_1" type="visual"/>
-        </geometry>
-      </visual>
-      <collision>
-        <origin xyz="0 0 ${visual_params}" rpy="${pi/2} 0 0"/>
-        <geometry>
-          <xacro:get_mesh name="wrist_1" type="collision"/>
-        </geometry>
-      </collision>
-      <xacro:cylinder_inertial radius="${wrist_1_inertia_radius}" length="${wrist_1_inertia_length}"  mass="${wrist_1_mass}">
-        <origin xyz="0 0 0" rpy="0 0 0" />
-      </xacro:cylinder_inertial>
-    </link>
-    <link name="${tf_prefix}wrist_2_link">
-	  <xacro:get_visual_params name="wrist_2" type="visual_offset"/>
-      <visual>
-        <origin xyz="0 0 ${visual_params}" rpy="0 0 0"/>
-        <geometry>
-          <xacro:get_mesh name="wrist_2" type="visual"/>
-        </geometry>
-      </visual>
-      <collision>
-        <origin xyz="0 0 ${visual_params}" rpy="0 0 0"/>
-        <geometry>
-          <xacro:get_mesh name="wrist_2" type="collision"/>
-        </geometry>
-      </collision>
-      <xacro:cylinder_inertial radius="${wrist_2_inertia_radius}" length="${wrist_2_inertia_length}"  mass="${wrist_2_mass}">
-        <origin xyz="0 0 0" rpy="0 0 0" />
-      </xacro:cylinder_inertial>
-    </link>
-    <link name="${tf_prefix}wrist_3_link">
-	  <xacro:get_visual_params name="wrist_3" type="visual_offset"/>
-      <visual>
-        <origin xyz="0 0 ${visual_params}" rpy="${pi/2} 0 0"/>
-        <geometry>
-          <xacro:get_mesh name="wrist_3" type="visual"/>
-        </geometry>
-      </visual>
-      <collision>
-        <origin xyz="0 0 ${visual_params}" rpy="${pi/2} 0 0"/>
-        <geometry>
-          <xacro:get_mesh name="wrist_3" type="collision"/>
-        </geometry>
-      </collision>
-      <xacro:cylinder_inertial radius="${wrist_3_inertia_radius}" length="${wrist_3_inertia_length}"  mass="${wrist_3_mass}">
-        <origin xyz="0.0 0.0 ${-0.5 * wrist_3_inertia_length}" rpy="0 0 0" />
-      </xacro:cylinder_inertial>
-    </link>
-    <!-- base_joint fixes base_link to the environment -->
-    <joint name="${tf_prefix}base_joint" type="fixed">
-      <xacro:insert_block name="origin" />
-      <parent link="${parent}" />
-      <child link="${tf_prefix}base_link" />
-    </joint>
-    <!-- joints - main serial chain -->
-    <joint name="${tf_prefix}base_link-base_link_inertia" type="fixed">
-      <parent link="${tf_prefix}base_link" />
-      <child link="${tf_prefix}base_link_inertia" />
-      <!-- 'base_link' is REP-103 aligned (so X+ forward), while the internal
+  >
+  <!-- Load configuration data from the provided .yaml files -->
+  <xacro:read_model_data
+    joint_limits_parameters_file="${joint_limits_parameters_file}"
+    kinematics_parameters_file="${kinematics_parameters_file}"
+    physical_parameters_file="${physical_parameters_file}"
+    visual_parameters_file="${visual_parameters_file}"
+    force_abs_paths="${sim_gazebo or sim_ignition}" />
+  <!-- ros2 control include -->
+  <xacro:include filename="$(find ur_description)/urdf/ur.ros2_control.xacro" />
+  <!-- ros2 control instance -->
+  <xacro:ur_ros2_control
+    name="${name}"
+    use_fake_hardware="${use_fake_hardware}"
+    initial_positions="${initial_positions}"
+    fake_sensor_commands="${fake_sensor_commands}"
+    headless_mode="${headless_mode}"
+    sim_gazebo="${sim_gazebo}"
+    sim_ignition="${sim_ignition}"
+    script_filename="${script_filename}"
+    output_recipe_filename="${output_recipe_filename}"
+    input_recipe_filename="${input_recipe_filename}"
+    tf_prefix="${tf_prefix}"
+    hash_kinematics="${kinematics_hash}"
+    robot_ip="${robot_ip}"
+    use_tool_communication="${use_tool_communication}"
+    tool_voltage="${tool_voltage}"
+    tool_parity="${tool_parity}"
+    tool_baud_rate="${tool_baud_rate}"
+    tool_stop_bits="${tool_stop_bits}"
+    tool_rx_idle_chars="${tool_rx_idle_chars}"
+    tool_tx_idle_chars="${tool_tx_idle_chars}"
+    tool_device_name="${tool_device_name}"
+    tool_tcp_port="${tool_tcp_port}"
+    reverse_port="${reverse_port}"
+    script_sender_port="${script_sender_port}"
+    reverse_ip="${reverse_ip}"
+    script_command_port="${script_command_port}"
+    trajectory_port="${trajectory_port}"
+    non_blocking_read="${non_blocking_read}"
+    keep_alive_count="${keep_alive_count}"
+  />
+  <!-- Add URDF transmission elements (for ros_control) -->
+  <!--<xacro:ur_arm_transmission
+    prefix="${prefix}" hw_interface="${transmission_hw_interface}" />-->
+  <!-- Placeholder for ros2_control transmission which don't yet exist -->
+  <!-- links -  main serial chain -->
+  <link name="${tf_prefix}base_link" />
+  <link name="${tf_prefix}base_link_inertia">
+    <visual>
+      <origin xyz="0 0 0" rpy="0 0 ${pi}" />
+      <geometry>
+        <xacro:get_mesh name="base" type="visual" />
+      </geometry>
+    </visual>
+    <collision>
+      <origin xyz="0 0 0" rpy="0 0 ${pi}" />
+      <geometry>
+        <xacro:get_mesh name="base" type="collision" />
+      </geometry>
+    </collision>
+    <xacro:cylinder_inertial radius="${base_inertia_radius}" length="${base_inertia_length}"
+      mass="${base_mass}">
+      <origin xyz="0 0 0" rpy="0 0 0" />
+    </xacro:cylinder_inertial>
+  </link>
+  <link name="${tf_prefix}shoulder_link">
+    <visual>
+      <origin xyz="0 0 0" rpy="0 0 ${pi}" />
+      <geometry>
+        <xacro:get_mesh name="shoulder" type="visual" />
+      </geometry>
+    </visual>
+    <collision>
+      <origin xyz="0 0 0" rpy="0 0 ${pi}" />
+      <geometry>
+        <xacro:get_mesh name="shoulder" type="collision" />
+      </geometry>
+    </collision>
+    <xacro:cylinder_inertial radius="${shoulder_inertia_radius}"
+      length="${shoulder_inertia_length}" mass="${shoulder_mass}">
+      <origin xyz="0 0 0" rpy="0 0 0" />
+    </xacro:cylinder_inertial>
+  </link>
+  <link name="${tf_prefix}upper_arm_link">
+    <visual>
+      <origin xyz="0 0 ${shoulder_offset}" rpy="${pi/2} 0 ${-pi/2}" />
+      <geometry>
+        <xacro:get_mesh name="upper_arm" type="visual" />
+      </geometry>
+    </visual>
+    <collision>
+      <origin xyz="0 0 ${shoulder_offset}" rpy="${pi/2} 0 ${-pi/2}" />
+      <geometry>
+        <xacro:get_mesh name="upper_arm" type="collision" />
+      </geometry>
+    </collision>
+    <xacro:cylinder_inertial radius="${upperarm_inertia_radius}"
+      length="${upperarm_inertia_length}" mass="${upper_arm_mass}">
+      <origin xyz="${-0.5 * upperarm_inertia_length} 0.0 ${upper_arm_inertia_offset}"
+        rpy="0 ${pi/2} 0" />
+    </xacro:cylinder_inertial>
+  </link>
+  <link name="${tf_prefix}forearm_link">
+    <visual>
+      <origin xyz="0 0 ${elbow_offset}" rpy="${pi/2} 0 ${-pi/2}" />
+      <geometry>
+        <xacro:get_mesh name="forearm" type="visual" />
+      </geometry>
+    </visual>
+    <collision>
+      <origin xyz="0 0 ${elbow_offset}" rpy="${pi/2} 0 ${-pi/2}" />
+      <geometry>
+        <xacro:get_mesh name="forearm" type="collision" />
+      </geometry>
+    </collision>
+    <xacro:cylinder_inertial radius="${forearm_inertia_radius}" length="${forearm_inertia_length}"
+      mass="${forearm_mass}">
+      <origin xyz="${-0.5 * forearm_inertia_length} 0.0 ${elbow_offset}" rpy="0 ${pi/2} 0" />
+    </xacro:cylinder_inertial>
+  </link>
+  <link name="${tf_prefix}wrist_1_link">
+    <xacro:get_visual_params name="wrist_1" type="visual_offset" />
+    <visual>
+      <origin xyz="0 0 ${visual_params}" rpy="${pi/2} 0 0" />
+      <geometry>
+        <xacro:get_mesh name="wrist_1" type="visual" />
+      </geometry>
+    </visual>
+    <collision>
+      <origin xyz="0 0 ${visual_params}" rpy="${pi/2} 0 0" />
+      <geometry>
+        <xacro:get_mesh name="wrist_1" type="collision" />
+      </geometry>
+    </collision>
+    <xacro:cylinder_inertial radius="${wrist_1_inertia_radius}" length="${wrist_1_inertia_length}"
+      mass="${wrist_1_mass}">
+      <origin xyz="0 0 0" rpy="0 0 0" />
+    </xacro:cylinder_inertial>
+  </link>
+  <link name="${tf_prefix}wrist_2_link">
+    <xacro:get_visual_params name="wrist_2" type="visual_offset" />
+    <visual>
+      <origin xyz="0 0 ${visual_params}" rpy="0 0 0" />
+      <geometry>
+        <xacro:get_mesh name="wrist_2" type="visual" />
+      </geometry>
+    </visual>
+    <collision>
+      <origin xyz="0 0 ${visual_params}" rpy="0 0 0" />
+      <geometry>
+        <xacro:get_mesh name="wrist_2" type="collision" />
+      </geometry>
+    </collision>
+    <xacro:cylinder_inertial radius="${wrist_2_inertia_radius}" length="${wrist_2_inertia_length}"
+      mass="${wrist_2_mass}">
+      <origin xyz="0 0 0" rpy="0 0 0" />
+    </xacro:cylinder_inertial>
+  </link>
+  <link name="${tf_prefix}wrist_3_link">
+    <xacro:get_visual_params name="wrist_3" type="visual_offset" />
+    <visual>
+      <origin xyz="0 0 ${visual_params}" rpy="${pi/2} 0 0" />
+      <geometry>
+        <xacro:get_mesh name="wrist_3" type="visual" />
+      </geometry>
+    </visual>
+    <collision>
+      <origin xyz="0 0 ${visual_params}" rpy="${pi/2} 0 0" />
+      <geometry>
+        <xacro:get_mesh name="wrist_3" type="collision" />
+      </geometry>
+    </collision>
+    <xacro:cylinder_inertial radius="${wrist_3_inertia_radius}" length="${wrist_3_inertia_length}"
+      mass="${wrist_3_mass}">
+      <origin xyz="0.0 0.0 ${-0.5 * wrist_3_inertia_length}" rpy="0 0 0" />
+    </xacro:cylinder_inertial>
+  </link>
+  <!-- base_joint fixes base_link to the environment -->
+  <joint name="${tf_prefix}base_joint" type="fixed">
+    <xacro:insert_block name="origin" />
+    <parent link="${parent}" />
+    <child link="${tf_prefix}base_link" />
+  </joint>
+  <!-- joints - main serial chain -->
+  <joint name="${tf_prefix}base_link-base_link_inertia" type="fixed">
+    <parent link="${tf_prefix}base_link" />
+    <child link="${tf_prefix}base_link_inertia" />
+    <!-- 'base_link' is REP-103 aligned (so X+ forward), while the internal
            frames of the robot/controller have X+ pointing backwards.
            Use the joint between 'base_link' and 'base_link_inertia' (a dummy
            link/frame) to introduce the necessary rotation over Z (of pi rad).
       -->
-      <origin xyz="0 0 0" rpy="0 0 ${pi}" />
-    </joint>
-    <joint name="${tf_prefix}shoulder_pan_joint" type="revolute">
-      <parent link="${tf_prefix}base_link_inertia" />
-      <child link="${tf_prefix}shoulder_link" />
-      <origin xyz="${shoulder_x} ${shoulder_y} ${shoulder_z}" rpy="${shoulder_roll} ${shoulder_pitch} ${shoulder_yaw}" />
-      <axis xyz="0 0 1" />
-      <limit lower="${shoulder_pan_lower_limit}" upper="${shoulder_pan_upper_limit}"
-        effort="${shoulder_pan_effort_limit}" velocity="${shoulder_pan_velocity_limit}"/>
-      <xacro:if value="${safety_limits}">
-         <safety_controller soft_lower_limit="${shoulder_pan_lower_limit + safety_pos_margin}" soft_upper_limit="${shoulder_pan_upper_limit - safety_pos_margin}" k_position="${safety_k_position}" k_velocity="0.0"/>
-      </xacro:if>
-      <dynamics damping="0" friction="0"/>
-    </joint>
-    <joint name="${tf_prefix}shoulder_lift_joint" type="revolute">
-      <parent link="${tf_prefix}shoulder_link" />
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
Commit message: camera addeed

File: ur_ws/src/Universal_Robots_ROS2_Description/urdf/ur_macro.xacro (robot description, xacro)
@@ -442,8 +442,13 @@
   <xacro:arg name="camera_model" default="zed2" />
   <xacro:arg name="custom_baseline" default="0.0" />
+  <!-- <joint name="camera_support_joint2" type="fixed">
+    <parent link="camera_support" />
+    <child link="zed2_camera_link" />
+    <origin xyz="-0.081653 0.018797 0.0" rpy="-${pi/2} 0.0 ${pi/2}" />
+  </joint> -->
   <joint name="camera_support_joint2" type="fixed">
     <parent link="camera_support" />
     <child link="zed2_camera_link" />
-    <origin xyz="-0.081653 0.018797 0.0" rpy="-${pi/2} 0.0 ${pi/2}" />
+    <origin xyz="-0.081653 0.045 0.0" rpy="-${pi/2} 0.0 ${pi/2}" />
   </joint>
   <!-- If GNSS fusion is enabled the position of the antenna with respect to the camera mount point
@@ -480,10 +485,18 @@
   </joint>
   <link
-  name="probe">
+  name="probe_bota">
   </link>
   <joint name="probe_joint" type="fixed">
     <parent link="probe_mounting" />
+    <child link="probe_bota" />
+    <origin xyz="0.0 0.0 0.14" rpy="0.0 0.0 0.0" />
+  </joint>
+  <link
+  name="probe">
+  </link>
+  <joint name="ft_ur_joint" type="fixed">
+    <parent link="tool0" />
     <child link="probe" />
-    <origin xyz="0.0 0.0 0.14" rpy="0.0 0.0 0.0" />
+    <origin xyz="0.0 0.0 0.21" rpy="0.0 0.0 0.0" />
   </joint>
 </xacro:macro>

Commit message: DEMO WIRED

File: ur_ws/src/Universal_Robots_ROS2_Description/urdf/ur_macro.xacro (robot description, xacro)
@@ -447,9 +447,9 @@
     <origin xyz="-0.081653 0.018797 0.0" rpy="-${pi/2} 0.0 ${pi/2}" />
   </joint> -->
-  <joint name="camera_support_joint2" type="fixed">
+  <!-- <joint name="camera_support_joint2" type="fixed">
     <parent link="camera_support" />
     <child link="zed2_camera_link" />
     <origin xyz="-0.081653 0.045 0.0" rpy="-${pi/2} 0.0 ${pi/2}" />
-  </joint>
+  </joint> -->
   <!-- If GNSS fusion is enabled the position of the antenna with respect to the camera mount point
   is required -->
@@ -458,9 +458,9 @@
   <xacro:arg name="gnss_y" default="0.0" />
   <xacro:arg name="gnss_z" default="0.0" />
-  <xacro:include filename="$(find zed_wrapper)/urdf/zed_macro.urdf.xacro" />
+  <!-- <xacro:include filename="$(find zed_wrapper)/urdf/zed_macro.urdf.xacro" />
   <xacro:zed_camera name="$(arg camera_name)" model="$(arg camera_model)"
     custom_baseline="$(arg custom_baseline)" enable_gnss="$(arg enable_gnss)">
     <origin xyz="$(arg gnss_x) $(arg gnss_y) $(arg gnss_z)" rpy="0 0 0" />
-  </xacro:zed_camera>
+  </xacro:zed_camera> -->
   <!-- US probe model -->
   <link

Commit message: removed ft

File: ur_ws/src/Universal_Robots_ROS2_Description/urdf/ur_macro.xacro (robot description, xacro)
@@ -402,65 +402,4 @@
     <child link="${tf_prefix}tool0" />
   </joint>
-  <!-- force sensor urdf -->
-  <xacro:include filename="$(find rokubimini_description)/urdf/BFT_SENS_ECAT_M8.urdf.xacro" />
-  <!-- FT SENSOR-->
-  <xacro:BFT_SENS_ECAT_M8 prefix="ft_sensor0" />
-  <joint name="bota_ft_sensor" type="fixed">
-    <parent link="${tf_prefix}ft_frame" />
-    <child link="ft_sensor0_mounting" />
-    <origin xyz="0.0 0.0 0.0" rpy="${pi} 0.0 ${pi/2}" />
-  </joint>
-  <!-- CAMERA ATTACHMENT-->
-  <link
-    name="camera_support">
-    <visual>
-      <origin xyz="0 0 0" rpy="0 0 ${pi}" />
-      <geometry>
-        <mesh filename="package://ur_description/meshes/camera_support.stl"
-          scale="0.001 0.001 0.001" />
-      </geometry>
-      <material
-        name="">
-        <color
-          rgba="0.6902 0.61176 0.52941 1" />
-      </material>
-    </visual>
-  </link>
-  <joint name="camera_support_joint1" type="fixed">
-    <parent link="ft_sensor0_wrench" />
-    <child link="camera_support" />
-    <origin xyz="0.00 0.00 0.00" rpy="-${pi/2} ${pi} ${pi/4}" />
-  </joint>
-  <!-- ZED -->
-  <!--
-    Parameters:
-      - name: the camera's name.  should match the parameter sent to the launch file for this camera
-      - model: the type of camera, one of zed, zedm, zed2, zed2i, zedx, zedxm, virtual
-      - enable_gnss: if true enable the URDF link
-  -->
-  <xacro:arg name="camera_name" default="zed2" />
-  <xacro:arg name="camera_model" default="zed2" />
-  <xacro:arg name="custom_baseline" default="0.0" />
-  <!-- <joint name="camera_support_joint2" type="fixed">
-    <parent link="camera_support" />
-    <child link="zed2_camera_link" />
-    <origin xyz="-0.081653 0.018797 0.0" rpy="-${pi/2} 0.0 ${pi/2}" />
-  </joint> -->
-  <!-- <joint name="camera_support_joint2" type="fixed">
-    <parent link="camera_support" />
-    <child link="zed2_camera_link" />
-    <origin xyz="-0.081653 0.045 0.0" rpy="-${pi/2} 0.0 ${pi/2}" />
-  </joint> -->
-  <!-- If GNSS fusion is enabled the position of the antenna with respect to the camera mount point
-  is required -->
-  <xacro:arg name="enable_gnss" default="false" />
-  <xacro:arg name="gnss_x" default="0.0" />
-  <xacro:arg name="gnss_y" default="0.0" />
-  <xacro:arg name="gnss_z" default="0.0" />
-  <!-- <xacro:include filename="$(find zed_wrapper)/urdf/zed_macro.urdf.xacro" />
-  <xacro:zed_camera name="$(arg camera_name)" model="$(arg camera_model)"
-    custom_baseline="$(arg custom_baseline)" enable_gnss="$(arg enable_gnss)">
-    <origin xyz="$(arg gnss_x) $(arg gnss_y) $(arg gnss_z)" rpy="0 0 0" />
-  </xacro:zed_camera> -->
   <!-- US probe model -->
   <link
@@ -480,5 +419,5 @@
   </link>
   <joint name="tip_tool" type="fixed">
-    <parent link="ft_sensor0_wrench" />
+    <parent link="tool0" />
     <child link="probe_mounting" />
     <origin xyz="0.0 0.0 0.0" rpy="0.0 0.0 0.0" />
